File: ddr3.kicad_sch (KiCad schematic)
At the start: 52 parts, among them U10 TPS51200DRCR, U9 AS4C256M16D3

Commit message: Schematic Update
Parts:
- R54: Author Antmicro -> (none); License Apache-2.0 -> (none)
Other:
- note added: "DDR3"
- moved on the sheet: C61, C62, C63, C64, C65, C66, C67, C68, C69, C70, C78, C79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
