File: ethernet.kicad_sch (KiCad schematic)
At the start: 55 parts, among them J3 L834-1G1T-S7, U11 KSZ9031RNXCA, Y1 ABM8G-27.000MHZ-18-D2Y-T

Commit message: Schematic Update
Other:
- note added: "Ethernet"
- moved on the sheet: C102, C110, C111, C112, C113, C114, C115, C116, C117, C118, C119, C120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
