File: fpga-banks-13-16.kicad_sch (KiCad schematic)
At the start: 19 parts, among them U1 XC7A100T-FGG484, Y4 ECS-2520MV-130-BN-TR

Commit message: Schematic Update
Other:
- note added: "FPGA Banks 13 - 14"
- moved on the sheet: C193, C72, C73, C74, C75, C76, C77, C84, R93, R94, U1A, Y4
