File: fpga-unit-b.kicad_sch (KiCad schematic)
At the start: 15 parts, among them U1 XC7A100T-FGG484

Commit message: Schematic Update
Other:
- note added: "FPGA Banks 15 - 16"
- moved on the sheet: C72, C73, C74, C75, C76, C77, C84, U1B
