File: fpga-unit-c.kicad_sch (KiCad schematic)
At the start: 33 parts, among them J10 640456-3, J6 878311020, J9 640456-3, U1 XC7A100T-FGG484

Commit message: Schematic Update
Parts:
- R88: Author Antmicro -> (none); License Apache-2.0 -> (none)
Other:
- note added: "FPGA Banks 34 - 35; CFG"
- moved on the sheet: C59, C72, C73, C74, C75, C76, C77, C78, C79, C80, C81, C82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
