File: fpga-unit-d.kicad_sch (KiCad schematic)
At the start: 13 parts, among them J2 Bus_PCI_Express_x1, U1 XC7A100T-FGG484

Commit message: Schematic Update
Other:
- note added: "Multi Gigabit Transceiver - MGT Pins"
- moved on the sheet: C100, C101, C140, C141, C142, C143, C144, C145, C59, C92, J2, R68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
