File: fpga-unit-f.kicad_sch (KiCad schematic)
At the start: 30 parts, among them U1 XC7A100T-FGG484

Commit message: Schematic Update
Other:
- note added: "FPGA Power Supply"
- moved on the sheet: C1, C10, C11, C12, C13, C14, C15, C16, C17, C18, C19, C2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
