File: hdmi.kicad_sch (KiCad schematic)
At the start: 7 parts, among them J7 10029449-111RLF, U15 TPD4E05U06DQAR, U16 TPD4E05U06DQAR

Commit message: Schematic Update
Other:
- note added: "HDMI Interface"
Changed lines of the file:
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@@
     (stroke (width 0) (type default))
   )
-  (text "Differential pairs @100 Ohms\n" (at 234.95 33.655 0)
+  (text "Differential pairs @100 Ohms\n" (at 217.17 137.16 0)
     (effects (font (size 1.27 1.27)) (justify left bottom))
   )
+  (text "HDMI Interface\n" (at 34.925 46.355 0)
+    (effects (font (size 7 7) (thickness 1.4) bold) (justify left bottom))
+  )
   (global_label "HDMI_CEC" (shape input) (at 77.47 93.98 180) (fields_autoplaced)
