File: power-supply.kicad_sch (KiCad schematic)
At the start: 81 parts, among them J1 DCJ200-10-A-XX-K_REVA, U2 TPS62823DLCT, U3 LM3881MMX/NOPB, U4 TPS62823DLCT, U6 TPS54561DPRR

Commit message: Schematic Update
Parts:
- R108, R110, R112, R113, R21, R7, R91, R92: Author Antmicro -> (none); License Apache-2.0 -> (none)
Other:
- note added: "12V Power Supply Downconverting"
- moved on the sheet: C30, C31, C32, C33, C34, C35, C39, C40, C41, C42, C43, C44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
