File: qspi_flash.kicad_sch (KiCad schematic)
At the start: 8 parts, among them IC1 MT25QL512ABB8ESF-0AAT

Commit message: Schematic Update
Other:
- note added: "FLASH Memory"
- moved on the sheet: C146, IC1, R70, R72, R74, R76, R78, R79
