File: usb.kicad_sch (KiCad schematic)
At the start: 50 parts, among them IC2 TPD2E009DBZR, J4 10118192-0002LF, J5 USB-A1VSB6, U12 FT4232H-56Q-TRAY, U13 USB3300-EZK, U14 SP3011-06UTG, Y2 ABM8G-12.000MHZ-18-D2Y-T, Y3 ABM8-24.000MHZ-B2-T

Commit message: Schematic Update
Other:
- moved on the sheet: C149, C150, C151, C152, C153, C154, C155, C156, C157, C158, C159, C160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
